File: DMH_Sequencer_PANEL/DMH_Sequencer_PANEL.kicad_sch (KiCad schematic)
At the start: 124 parts, among them J0 Panel_GND_Solder_Wire_Pad

Commit message: Added Gate out and Reset in for 9 to 16
Parts:
- added H116: Rst 1-8, SynthStuff:Jack_6.35mm_Cutout_v3, symbol SynthStuff:MountingHole_Jack6.35mm_v2
- H73: value Clock Speed -> Clock
- H88: value Gate -> Gate 1-8
- H89: value 9-16 -> Gate 9-16; now fitted
- H91: value Reset -> Rst 9-16
Connections:
- net GND: now also H116.1
Other:
- moved on the sheet: H92
Changed lines of the file:
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@@
 	)
 	(junction
+		(at 76.2 146.05)
+		(diameter 0)
+		(color 0 0 0 0)
+	)
+	(junction
 		(at 215.9 148.59)
 		(diameter 0)
@@
 	(wire
 		(pts
-			(xy 50.8 146.05) (xy 101.6 146.05)
+			(xy 50.8 146.05) (xy 76.2 146.05)
 		)
 		(stroke
@@
 	(wire
 		(pts
+			(xy 101.6 146.05) (xy 76.2 146.05)
+		)
+		(stroke
+			(width 0)
+			(type default)
+		)
+	)
+	(wire
+		(pts
 			(xy 139.7 107.95) (xy 114.3 107.95)
 		)
@@
 	(wire
 		(pts
-			(xy 101.6 143.51) (xy 101.6 146.05)
+			(xy 76.2 143.51) (xy 76.2 146.05)
 		)
 		(stroke
@@
 	(wire
 		(pts
+			(xy 101.6 143.51) (xy 101.6 146.05)
+		)
+		(stroke
+			(width 0)
+			(type default)
+		)
+	)
+	(wire
+		(pts
 			(xy 190.5 148.59) (xy 203.2 148.59)
 		)
@@
 			)
 		)
-		(property "Value" "Gate"
+		(property "Value" "Gate 1-8"
 			(at 27.94 127 90)
 			(effects
@@
 			)
 		)
-		(property "Value" "Reset"
+		(property "Value" "Rst 9-16"
 			(at 104.14 152.4 90)
 			(effects
@@
 	)
 	(symbol
+		(lib_id "SynthStuff:MountingHole_Jack6.35mm_v2")
+		(at 101.6 139.7 90)
+		(unit 1)
+		(exclude_from_sim no)
+		(in_bom no)
+		(on_board yes)
+		(dnp no)
+		(fields_autoplaced yes)
+		(property "Reference" "H116"
+			(at 104.14 137.1599 90)
+			(effects
+				(font
+					(size 1.27 1.27)
+				)
+				(justify right)
+			)
+		)
+		(property "Value" "Rst 1-8"
+			(at 104.14 139.7 90)
+			(effects
+				(font
+					(size 1.27 1.27)
+					(thickness 0.254)
+					(bold yes)
+					(italic yes)
+				)
+				(justify right)
+			)
+		)
+		(property "Footprint" "SynthStuff:Jack_6.35mm_Cutout_v3"
+			(at 101.6 139.7 0)
+			(effects
+				(font
+					(size 1.27 1.27)
+				)
+				(hide yes)
+			)
+		)
+		(property "Datasheet" "~"
+			(at 101.6 139.7 0)
+			(effects
+				(font
+					(size 1.27 1.27)
+				)
+				(hide yes)
+			)
+		)
+		(property "Description" "Jack 6.35mm"
+			(at 104.14 142.2399 90)
+			(effects
+				(font
+					(size 1.27 1.27)
+				)
+				(justify right)
+			)
+		)
+		(pin "1"
+		)
+		(instances
+			(project "DMH_Sequencer_PANEL"
+				(path "/a552705f-a9fe-462e-9913-5cfcc08b233c"
+					(reference "H116")
+					(unit 1)
+				)
+			)
+		)
+	)
+	(symbol
 		(lib_id "SynthStuff:MountingHole_ToggleSwitch")
 		(at 50.8 76.2 0)
@@
 		(exclude_from_sim no)
 		(in_bom no)
-		(on_board no)
-		(dnp yes)
+		(on_board yes)
+		(dnp no)
 		(fields_autoplaced yes)
 		(property "Reference" "H89"
@@
 			)
 		)
-		(property "Value" "9-16"
+		(property "Value" "Gate 9-16"
 			(at 53.34 127 90)
 			(effects
@@
 			)
 		)
-		(property "Value" "Clock Speed"
+		(property "Value" "Clock"
 			(at 27.94 25.4 0)
 			(effects
@@
 	(symbol
 		(lib_id "SynthStuff:MountingHole_Jack6.35mm_v2")
-		(at 101.6 139.7 90)
+		(at 76.2 139.7 90)
 		(unit 1)
 		(exclude_from_sim no)
@@
 		(fields_autoplaced yes)
 		(property "Reference" "H92"
-			(at 104.14 137.1599 90)
+			(at 78.74 137.1599 90)
 			(effects
 				(font
@@
 		)
 		(property "Value" "Transp"
-			(at 104.14 139.7 90)
+			(at 78.74 139.7 90)
 			(effects
 				(font
@@
 		)
 		(property "Footprint" "SynthStuff:Jack_6.35mm_Cutout_v3"
-			(at 101.6 139.7 0)
+			(at 76.2 139.7 0)
 			(effects
 				(font
@@
 		)
 		(property "Datasheet" "~"
-			(at 101.6 139.7 0)
+			(at 76.2 139.7 0)
 			(effects
 				(font
@@
 		)
 		(property "Description" "Jack 6.35mm"
-			(at 104.14 142.2399 90)
+			(at 78.74 142.2399 90)
 			(effects
 				(font
